Commit message: Add use_gazebo param to fairino xacro; raise effort limits for Gazebo sim (#3)
* Add use_gazebo param to fairino xacro; raise effort limits for Gazebo sim

fairino.ros2_control.xacro:
- Add use_gazebo:=false param alongside use_fake_hardware
- Three-way plugin selection: GazeboSimSystem (use_gazebo), mock_components
  (use_fake_hardware), FairinoHardwareInterface (real robot)
- Fixes the revert in 60862be: GazeboSimSystem was tied to use_fake_hardware
  which also covers MoveIt fake-hardware mode (no Gazebo running)

fairino20_v6.urdf:
- j1-j3 effort limit: 150 -> 1000 Nm
- j4-j6 effort limit: 28 -> 500 Nm
- Prevents arm gravitational sag under gz_ros2_control position control

Co-Authored-By: Claude Sonnet 4.6 <noreply@anthropic.com>

* Add joint damping for Gazebo simulation stability

j1-j3: 100 N·m·s/rad, j4-j6: 30 N·m·s/rad — prevents gravity-induced
oscillation when using GazeboSimSystem position→velocity control.

Co-Authored-By: Claude Sonnet 4.6 <noreply@anthropic.com>

---------

Co-authored-by: Claude Sonnet 4.6 <noreply@anthropic.com>

File: fairino_description/urdf/fairino.ros2_control.xacro (robot description, xacro)
@@ -3,5 +3,5 @@
   <xacro:macro
     name="fairino_ros2_control"
-    params="name fairino_file use_fake_hardware:=false"
+    params="name fairino_file use_fake_hardware:=false use_gazebo:=false"
   >
     <xacro:property name="ip_address" value="${xacro.load_yaml(fairino_file)['ip_address']}" />
@@ -9,10 +9,15 @@
     <ros2_control name="${name}" type="system">
       <hardware>
-        <xacro:if value="${use_fake_hardware}">
-          <plugin>mock_components/GenericSystem</plugin>
+        <xacro:if value="${use_gazebo}">
+          <plugin>gz_ros2_control/GazeboSimSystem</plugin>
         </xacro:if>
-        <xacro:unless value="${use_fake_hardware}">
-          <plugin>fairino_hardware/FairinoHardwareInterface</plugin>
-          <param name="ip_address">${ip_address}</param>
+        <xacro:unless value="${use_gazebo}">
+          <xacro:if value="${use_fake_hardware}">
+            <plugin>mock_components/GenericSystem</plugin>
+          </xacro:if>
+          <xacro:unless value="${use_fake_hardware}">
+            <plugin>fairino_hardware/FairinoHardwareInterface</plugin>
+            <param name="ip_address">${ip_address}</param>
+          </xacro:unless>
         </xacro:unless>
       </hardware>

File: fairino_description/urdf/fairino20_v6.urdf (robot description, URDF)
Before this commit: robot fairino20_v6_robot, 7 links, 6 joints
Joints:
- joint j1: limit lower=-3.0543 upper=3.0543 effort=150 velocity=3.15 -> lower=-3.0543 upper=3.0543 effort=1000 velocity=3.15
- joint j2: limit lower=-4.6251 upper=1.4835 effort=150 velocity=3.15 -> lower=-4.6251 upper=1.4835 effort=1000 velocity=3.15
- joint j3: limit lower=-2.8274 upper=2.8274 effort=150 velocity=3.15 -> lower=-2.8274 upper=2.8274 effort=1000 velocity=3.15
- joint j4: limit lower=-4.6251 upper=1.4835 effort=28 velocity=3.2 -> lower=-4.6251 upper=1.4835 effort=500 velocity=3.2
- joint j5: limit lower=-3.0543 upper=3.0543 effort=28 velocity=3.2 -> lower=-3.0543 upper=3.0543 effort=500 velocity=3.2
- joint j6: limit lower=-3.0543 upper=3.0543 effort=28 velocity=3.2 -> lower=-3.0543 upper=3.0543 effort=500 velocity=3.2
