Commit message: FR10: joint position and soft limits from the datasheet
j3 hard limit was ±162°; the FR10 datasheet gives ±160°. Soft limits
were a ±175° placeholder on every joint, which clipped j2/j4 (-265°/+85°)
and exceeded the j3 range. Soft limits now follow the fairino20_v6
pattern: hard limit minus 2° on each side.

Source: https://www.frtech.fr/FR/3.html (FR10 axis movement table).

Co-Authored-By: Claude Opus 5.5 <noreply@anthropic.com>
Claude-Session: https://claude.ai/code/session_017dQcz8TS8CximyEnUgEG2t

File: fairino_description/urdf/fairino10_v6.urdf (robot description, URDF)
Before this commit: robot fairino10_v6_robot, 7 links, 6 joints
Joints:
- joint j3: limit lower=-2.8274 upper=2.8274 effort=150 velocity=3.15 -> lower=-2.7925 upper=2.7925 effort=150 velocity=3.15

Commit message: FR10: j3 limits match fairino20_v6 (hard ±162°, soft ±160°)
The datasheet gives ±160° for j3 on both FR10 and FR20. #6 set FR10 to
hard ±160° / soft ±158°, while fairino20_v6 keeps the vendor hard ±162° /
soft ±160°. MoveIt plans on soft limits, so the elbow differed by 2° between
arms. Match FR20 so both arms carry identical position and soft limits; the
planning limit stays at the datasheet ±160°.

Co-Authored-By: Claude Opus 5.5 <noreply@anthropic.com>
Claude-Session: https://claude.ai/code/session_017dQcz8TS8CximyEnUgEG2t

File: fairino_description/urdf/fairino10_v6.urdf (robot description, URDF)
Before this commit: robot fairino10_v6_robot, 7 links, 6 joints
Joints:
- joint j3: limit lower=-2.7925 upper=2.7925 effort=150 velocity=3.15 -> lower=-2.8274 upper=2.8274 effort=150 velocity=3.15

Commit message: FR10, FR20: joint limits and velocities from the Fairino basic parameters table
Table 2.1-1 lists the controller's soft and hard working ranges and max
joint speeds. URDF <limit> now holds the controller hard limit
(±179°, +89/−269°, j3 ±162°) and safety_controller holds the controller
soft limit (±175°, +85/−265°, j3 ±160°). Velocities: 120°/s on FR10
j1–j2 and FR20 j1–j3, 180°/s elsewhere, in both the URDFs and the
moveit2_config joint_limits.yaml.

Source: https://fairino-doc-en.readthedocs.io/latest/CobotsManual/robot_brief_introduction.html#basic-parameters

Co-Authored-By: Claude Opus 5.5 <noreply@anthropic.com>
Claude-Session: https://claude.ai/code/session_017dQcz8TS8CximyEnUgEG2t

File: fairino_description/urdf/fairino10_v6.urdf (robot description, URDF)
Before this commit: robot fairino10_v6_robot, 7 links, 6 joints
Joints:
- joint j1: limit lower=-3.0543 upper=3.0543 effort=150 velocity=3.15 -> lower=-3.1241 upper=3.1241 effort=150 velocity=2.0944
- joint j2: limit lower=-4.6251 upper=1.4835 effort=150 velocity=3.15 -> lower=-4.6949 upper=1.5533 effort=150 velocity=2.0944
- joint j3: limit lower=-2.8274 upper=2.8274 effort=150 velocity=3.15 -> lower=-2.8274 upper=2.8274 effort=150 velocity=3.1416
- joint j4: limit lower=-4.6251 upper=1.4835 effort=28 velocity=3.2 -> lower=-4.6949 upper=1.5533 effort=28 velocity=3.1416
- joint j5: limit lower=-3.0543 upper=3.0543 effort=28 velocity=3.2 -> lower=-3.1241 upper=3.1241 effort=28 velocity=3.1416
- joint j6: limit lower=-3.0543 upper=3.0543 effort=28 velocity=3.2 -> lower=-3.1241 upper=3.1241 effort=28 velocity=3.1416

File: fairino_description/urdf/fairino20_v6.urdf (robot description, URDF)
Before this commit: robot fairino20_v6_robot, 7 links, 6 joints
Joints:
- joint j1: limit lower=-3.0543 upper=3.0543 effort=1000 velocity=3.15 -> lower=-3.1241 upper=3.1241 effort=1000 velocity=2.0944
- joint j2: limit lower=-4.6251 upper=1.4835 effort=1000 velocity=3.15 -> lower=-4.6949 upper=1.5533 effort=1000 velocity=2.0944
- joint j3: limit lower=-2.8274 upper=2.8274 effort=1000 velocity=3.15 -> lower=-2.8274 upper=2.8274 effort=1000 velocity=2.0944
- joint j4: limit lower=-4.6251 upper=1.4835 effort=500 velocity=3.2 -> lower=-4.6949 upper=1.5533 effort=500 velocity=3.1416
- joint j5: limit lower=-3.0543 upper=3.0543 effort=500 velocity=3.2 -> lower=-3.1241 upper=3.1241 effort=500 velocity=3.1416
- joint j6: limit lower=-3.0543 upper=3.0543 effort=500 velocity=3.2 -> lower=-3.1241 upper=3.1241 effort=500 velocity=3.1416
